Commit message: Add RM3100 and CURT to the setup and fix mapir mapping device port

File: ros2_ws/curt_description/urdf/robot.urdf.xacro (robot description, xacro)
@@ -12,5 +12,5 @@
   <xacro:include filename="properties.xacro" />
   <!-- Include sensors -->
-  <!-- <xacro:include filename="sensors.xacro" /> -->
+  <xacro:include filename="sensors.xacro" />
   <link name="base_link" />
   <!-- Chassis link at same position as base_link, as root is not allowed to have inertial
@@ -171,161 +171,3 @@
     <xacro:include filename="gazebo.xacro" />
   </xacro:if>
-  <!-- OUSTER TOWER VISUAL LINK -->
-  <!-- This link contains only the visual mesh for the ouster lidar -->
-  <link name="ouster_tower_visual">
-    <visual>
-      <origin xyz="0 0 0" rpy="0 0 0" />
-      <geometry>
-        <mesh filename="${mesh_prefix}meshes/Assembly_OS1.obj" />
-      </geometry>
-    </visual>
-    <inertial>
-      <mass value="1e-5"/>
-      <origin rpy="0 0 0" xyz="0.0 0 0.0"/>
-      <inertia ixx="1e-6" ixy="0" ixz="0" iyy="1e-6" iyz="0" izz="1e-6"/>
-    </inertial>
-  </link>
-  <!-- OUSTER TOWER VISUAL JOINT -->
-  <!-- This joint positions the visual mesh -->
-  <joint name="base_link_to_ouster_tower_visual" type="fixed">
-    <parent link="base_link" />
-    <child link="ouster_tower_visual" />
-    <origin xyz="-0.1105 0 0.204"
-            rpy="0 0 ${PI}" />
-  </joint>
-  <!-- CAMERA TOWER VISUAL LINK -->
-  <!-- This link contains only the visual mesh for all three cameras -->
-  <link name="cameras_tower_visual">
-    <visual>
-      <origin xyz="0 0 0" rpy="0 0 0" />
-      <geometry>
-        <mesh filename="${mesh_prefix}meshes/Assembly_Cameras.obj" />
-      </geometry>
-    </visual>
-    <inertial>
-      <mass value="1e-5"/>
-      <origin rpy="0 0 0" xyz="0.0 0 0.0"/>
-      <inertia ixx="1e-6" ixy="0" ixz="0" iyy="1e-6" iyz="0" izz="1e-6"/>
-    </inertial>
-  </link>
-  <!-- CAMERA TOWER VISUAL JOINT -->
-  <!-- This joint positions the visual mesh -->
-  <joint name="base_link_to_cameras_tower_visual" type="fixed">
-    <parent link="base_link" />
-    <child link="cameras_tower_visual" />
-    <origin xyz="-0.2407 0 0.204"
-            rpy="0 0 ${PI}" />
-  </joint>
-  <!-- ========================================== -->
-  <!-- OUSTER OS1 LINK TREE (CALIBRATED)          -->
-  <!-- base_link -> os_sensor -> (os_lidar, os_imu) -->
-  <!-- ========================================== -->
-  <!-- OS_SENSOR LINK -->
-  <link name="os_sensor">
-    <inertial>
-      <mass value="1e-5"/>
-      <origin rpy="0 0 0" xyz="0.0 0 0.0"/>
-      <inertia ixx="1e-6" ixy="0" ixz="0" iyy="1e-6" iyz="0" izz="1e-6"/>
-    </inertial>
-  </link>
-  <!-- OS_SENSOR JOINT -->
-  <joint name="base_link_to_os_sensor" type="fixed">
-    <parent link="base_link" />
-    <child link="os_sensor" />
-    <origin xyz="-0.1105 0.0 0.404" rpy="0.0 0.0 0" />
-  </joint>
-  <!-- OS_LIDAR LINK -->
-  <link name="os_lidar">
-    <inertial>
-      <mass value="1e-5"/>
-      <origin rpy="0 0 0" xyz="0.0 0 0.0"/>
-      <inertia ixx="1e-6" ixy="0" ixz="0" iyy="1e-6" iyz="0" izz="1e-6"/>
-    </inertial>
-  </link>
-  <!-- OS_LIDAR JOINT -->
-  <joint name="os_sensor_to_os_lidar" type="fixed">
-    <parent link="os_sensor" />
-    <child link="os_lidar" />
-    <origin xyz="0.0 0.0 0.0" rpy="0.0 0.0 0.0" />
-  </joint>
-  <!-- OS_IMU LINK -->
-  <link name="os_imu">
-    <inertial>
-      <mass value="1e-5"/>
-      <origin rpy="0 0 0" xyz="0.0 0 0.0"/>
-      <inertia ixx="1e-6" ixy="0" ixz="0" iyy="1e-6" iyz="0" izz="1e-6"/>
-    </inertial>
-  </link>
-  <!-- OS_IMU JOINT -->
-  <joint name="os_sensor_to_os_imu" type="fixed">
-    <parent link="os_sensor" />
-    <child link="os_imu" />
-    <origin xyz="0.0 0.0 0.0" rpy="0.0 0.0 0.0" />
-  </joint>
-  <!-- ========================================== -->
-  <!-- REALSENSE LINK TREE (CALIBRATED)           -->
-  <!-- base_link -> camera_link -> camera_color_optical_frame -->
-  <!-- ========================================== -->
-  <!-- CAMERA_LINK (RealSense Physical Mount) -->
-  <link name="camera_link">
-    <collision>
-      <origin rpy="0 0 0" xyz="0.0 0 0.0"/>
-      <geometry>
-        <box size="0.09 0.03 0.035"/>
-      </geometry>
-    </collision>
-    <inertial>
-      <mass value="1e-5"/>
-      <origin rpy="0 0 0" xyz="0.0 0 0.0"/>
-      <inertia ixx="1e-6" ixy="0" ixz="0" iyy="1e-6" iyz="0" izz="1e-6"/>
-    </inertial>
-  </link>
-  <!-- CAMERA_LINK JOINT -->
-  <joint name="base_link_to_camera_link" type="fixed">
-    <parent link="base_link" />
-    <child link="camera_link" />
-    <origin xyz="0.0 0.0 0.0" rpy="0.0 0.0 ${PI}" />
-  </joint>
-  <!-- CAMERA_COLOR_OPTICAL_FRAME LINK -->
-  <!-- This is the actual optical frame for the RealSense color camera -->
-  <link name="camera_color_optical_frame">
-    <inertial>
-      <mass value="1e-5"/>
-      <origin rpy="0 0 0" xyz="0.0 0 0.0"/>
-      <inertia ixx="1e-6" ixy="0" ixz="0" iyy="1e-6" iyz="0" izz="1e-6"/>
-    </inertial>
-  </link>
-  <!-- CALIBRATED JOINT: os_lidar -> camera_color_optical_frame -->
-  <!-- This is the calibrated transform between the Ouster LiDAR and RealSense camera -->
-  <joint name="joint_os_lidar_to_camera_color_optical_frame" type="fixed">
-    <parent link="os_lidar" />
-    <child link="camera_color_optical_frame" />
-    <origin xyz="-0.07047971203783951 -0.043647424976414335 -0.11746556974885704"
-            rpy="-1.567434123604688 -0.021310026725099566 ${1.575724678749616}" />
-  </joint>
-  <!-- ========================================== -->
-  <!-- MAPIR SURVEY3 LINK TREE                    -->
-  <!-- base_link -> mapir_link                    -->
-  <!-- ========================================== -->
-  <!-- MAPIR_LINK (Survey3) -->
-  <link name="mapir_link">
-    <collision>
-      <origin rpy="0 0 0" xyz="0.0 0 0.0"/>
-      <geometry>
-        <box size="0.03 0.03 0.03"/>
-      </geometry>
-    </collision>
-    <inertial>
-      <mass value="1e-5"/>
-      <origin rpy="0 0 0" xyz="0.0 0 0.0"/>
-      <inertia ixx="1e-6" ixy="0" ixz="0" iyy="1e-6" iyz="0" izz="1e-6"/>
-    </inertial>
-  </link>
-  <!-- MAPIR_LINK JOINT -->
-  <joint name="joint_os_lidar_to_mapir_link" type="fixed">
-    <parent link="os_lidar" />
-    <child link="mapir_link" />
-    <origin xyz="-2.106662958227812 -0.12660079802004065 -0.4261798662202779"
-            rpy="-1.7155973620374017 0.03380963393293503 ${1.1839555185746582 + PI}" />
-  </joint>
 </robot>
