Commit message: Add scovox and explo_planner. Changed tf frames and namespaces to multi-robot

File: ros2_ws/src/curt_description/urdf/gazebo.xacro (robot description, xacro)
@@ -3,5 +3,5 @@
   <!-- Some properties -->
   <xacro:include filename="properties.xacro" />
-  <gazebo reference="base_link">
+  <gazebo reference="base_link_curt">
     <material>Gazebo/Grey</material>
   </gazebo>

File: ros2_ws/src/curt_description/urdf/robot.urdf.xacro (robot description, xacro)
@@ -13,5 +13,5 @@
   <!-- Include sensors -->
   <xacro:include filename="sensors.xacro" />
-  <link name="base_link" />
+  <link name="base_link_curt" />
   <!-- Chassis link at same position as base_link, as root is not allowed to have inertial
   information -->
@@ -40,5 +40,5 @@
   </link>
   <joint name="base_to_chassis" type="fixed">
-    <parent link="base_link" />
+    <parent link="base_link_curt" />
     <child link="chassis" />
   </joint>
@@ -68,5 +68,5 @@
   <joint name="front_right_motor" type="continuous">
     <origin xyz="0.25995 -0.258 -0.030204" rpy="0 0 0" />
-    <parent link="base_link" />
+    <parent link="base_link_curt" />
     <child link="front_right_wheel" />
     <axis xyz="0 1 0" />
@@ -99,5 +99,5 @@
   <joint name="front_left_motor" type="continuous">
     <origin xyz="0.25995 0.258 -0.030204" rpy="0 0 0" />
-    <parent link="base_link" />
+    <parent link="base_link_curt" />
     <child link="front_left_wheel" />
     <axis xyz="0 1 0" />
@@ -130,5 +130,5 @@
   <joint name="back_right_motor" type="continuous">
     <origin xyz="-0.26 -0.258 -0.022755" rpy="0 0 0" />
-    <parent link="base_link" />
+    <parent link="base_link_curt" />
     <child link="back_right_wheel" />
     <axis xyz="0 1 0" />
@@ -161,5 +161,5 @@
   <joint name="back_left_motor" type="continuous">
     <origin xyz="-0.26 0.258 -0.022755" rpy="0 0 0" />
-    <parent link="base_link" />
+    <parent link="base_link_curt" />
     <child link="back_left_wheel" />
     <axis xyz="0 1 0" />

File: ros2_ws/src/curt_description/urdf/sensors.xacro (robot description, xacro)
@@ -13,23 +13,23 @@
   <!-- LPResearch CANAL3 IMU -->
   <joint name="base_link_to_imu" type="fixed">
-    <parent link="base_link" />
-    <child link="imu_link" />
+    <parent link="base_link_curt" />
+    <child link="imu_curt" />
     <origin xyz="0.062 0.0 0.015" rpy="0.0 0.0 -${pi/2}" />
   </joint>
-  <link name="imu_link" />
+  <link name="imu_curt" />
   <!-- RM3100 MAG -->
   <joint name="base_link_to_mag" type="fixed">
-    <parent link="base_link" />
-    <child link="mag" />
+    <parent link="base_link_curt" />
+    <child link="mag_curt" />
     <origin xyz="-0.2 0.0 0.204" rpy="0.0 0.0 ${pi/2}" />
   </joint>
-  <link name="mag" />
+  <link name="mag_curt" />
   <!-- Emlid Antenna -->
   <joint name="base_link_to_gps" type="fixed">
-    <parent link="base_link" />
-    <child link="gps" />
+    <parent link="base_link_curt" />
+    <child link="gps_curt" />
     <origin xyz="-0.25 0.11 0.204" rpy="0.0 0.0 0.0" />
   </joint>
-  <link name="gps" />
+  <link name="gps_curt" />
   <!-- OUSTER TOWER VISUAL LINK -->
   <!-- This link contains only the visual mesh for the ouster lidar -->
@@ -50,5 +50,5 @@
   <!-- This joint positions the visual mesh -->
   <joint name="base_link_to_ouster_tower_visual" type="fixed">
-    <parent link="base_link" />
+    <parent link="base_link_curt" />
     <child link="ouster_tower_visual" />
     <origin xyz="0.1105 0 0.204"
@@ -73,5 +73,5 @@
   <!-- This joint positions the visual mesh -->
   <joint name="base_link_to_cameras_tower_visual" type="fixed">
-    <parent link="base_link" />
+    <parent link="base_link_curt" />
     <child link="cameras_tower_visual" />
     <origin xyz="0.2407 0 0.204"
@@ -92,5 +92,5 @@
   <!-- OS_SENSOR JOINT -->
   <joint name="base_link_to_os_sensor" type="fixed">
-    <parent link="base_link" />
+    <parent link="base_link_curt" />
     <child link="os_sensor" />
     <origin xyz="0.1105 0.0 0.404" rpy="0.0 0.0 ${pi}" />
@@ -164,5 +164,5 @@
   <!-- ========================================== -->
   <!-- CAMERA_LINK (RealSense Physical Mount) -->
-  <link name="camera_link">
+  <link name="camera_curt_link">
     <collision>
       <origin rpy="0 0 0" xyz="0.0 0 0.0" />
@@ -179,11 +179,11 @@
   <!-- CAMERA_LINK JOINT -->
   <joint name="base_link_to_camera_link" type="fixed">
-    <parent link="base_link" />
-    <child link="camera_link" />
+    <parent link="base_link_curt" />
+    <child link="camera_curt_link" />
     <origin xyz="0.0 0.0 0.0" rpy="0.0 0.0 0.0" />
   </joint>
   <!-- CAMERA_COLOR_OPTICAL_FRAME LINK -->
   <!-- This is the actual optical frame for the RealSense color camera -->
-  <link name="camera_color_optical_frame">
+  <link name="camera_curt_color_optical_frame">
     <inertial>
       <mass value="1e-5" />
@@ -202,5 +202,5 @@
   <joint name="joint_os_lidar_to_camera_color_optical_frame" type="fixed">
     <parent link="os_lidar" />
-    <child link="camera_color_optical_frame" />
+    <child link="camera_curt_color_optical_frame" />
     <origin xyz="-0.16017594021604675 -0.04929723933704603 -0.12489075373962405" rpy="-1.5727906392966173 -0.027026586713933824 1.5723834999258628" />
   </joint>
